File: hardware/audio_shield_prod/audio_shield.sch (KiCad schematic (older format))
At the start: 48 parts, among them J1 CONN_10_LEFT, J2 CONN_10_RIGHT, J3 mic_connector, J4 mic_connector, J44 Conn_01x01_Female, J45 Conn_01x01_Female, J46 Conn_01x01_Female, J47 Conn_01x01_Female, J48 STLINK-V3MINI Placeholder, J5 mic_connector, J6 mic_connector, J7 mic_connector, J8 mic_connector, J9 SWD_TC2030

Commit message: annotation added
Parts:
- gave numbers to parts that had none: 1
Changed lines of the file:
@@
 $EndComp
 $Comp
-L audio_shield:DS28E05P U?
+L audio_shield:DS28E05P U2
 U 1 1 5F3EF92F
 P 1600 6750
-F 0 "U?" H 1600 6915 50  0000 C CNN
+F 0 "U2" H 1600 6915 50  0000 C CNN
 F 1 "DS28E05P" H 1600 6824 50  0000 C CNN
 F 2 "Package_SO_J-Lead:TSOC-6_3.76x3.94mm_P1.27mm" H 1600 6800 50  0001 C CNN
@@
 EEPROM for deck identification
 $Comp
-L power:GND #PWR?
+L power:GND #PWR0129
 U 1 1 5F4170B9
 P 1200 6850
-F 0 "#PWR?" H 1200 6600 50  0001 C CNN
+F 0 "#PWR0129" H 1200 6600 50  0001 C CNN
 F 1 "GND" H 1205 6677 50  0000 C CNN
 F 2 "" H 1200 6850 50  0001 C CNN
