File: hardware/audio_shield_prod/audio_shield.sch (KiCad schematic (older format))
At the start: 48 parts, among them J1 CONN_10_LEFT, J2 CONN_10_RIGHT, J3 mic_connector, J4 mic_connector, J44 Conn_01x01_Female, J45 Conn_01x01_Female, J46 Conn_01x01_Female, J47 Conn_01x01_Female, J48 STLINK-V3MINI Placeholder, J5 mic_connector, J6 mic_connector, J7 mic_connector, J8 mic_connector, J9 SWD_TC2030, U2 DS28E05P

Commit message: added comment
Other:
- note added: "I2C adress 47\n"
Changed lines of the file:
@@
 Wire Wire Line
 	950  6950 1300 6950
+Text Notes 700  3200 0    50   ~ 0
+I2C adress 47\n
 $EndSCHEMATC
