File: hardware/audio_shield_prod/stm32f446re.sch (KiCad schematic (older format))
At the start: 12 parts, among them U1 STM32F446RETx

Commit message: Edit component attribute for eurocircuit manufacturing
Parts:
- R1: Description (none) -> Thick film resistor 0.1W 1%
- U1: Description (none) -> Microcontrôleur 32bit 512KB LQFP-64
Changed lines of the file:
@@
 F 5 "300-56-687" H 4450 2250 50  0001 C CNN "Supplier ref."
 F 6 "0.0084" H 4450 2250 50  0001 C CNN "Price"
+F 7 "Thick film resistor 0.1W 1%" H 4450 2250 50  0001 C CNN "Description"
 	1    4450 2250
 	1    0    0    -1
@@
 F 5 "301-70-759" H 5600 3250 50  0001 C CNN "Supplier ref."
 F 6 "8.63" H 5600 3250 50  0001 C CNN "Price"
+F 7 "Microcontrôleur 32bit 512KB LQFP-64" H 5600 3250 50  0001 C CNN "Description"
 	1    5600 3250
 	1    0    0    -1
