File: hardware/audio_shield_prod/audio_shield.kicad_pcb (KiCad board)
At the start: 2 copper layers, 133 x 133 mm, 129 parts, among them J1 CONN_10_LEFT, J10 Conn_01x02_Male, J11 Conn_01x02_Male, J12 Conn_01x02_Male, J13 Conn_01x02_Male, J14 Conn_01x02_Male, J15 Conn_01x02_Male, J16 Conn_01x02_Male, J17 Conn_01x02_Male, J18 Conn_01x02_Male, J19 Conn_01x02_Male, J2 CONN_10_RIGHT, J20 Conn_01x02_Male, J21 Conn_01x02_Male, J22 Conn_01x02_Male, J23 Conn_01x02_Male, J24 Conn_01x02_Male, J25 Conn_01x02_Male, J26 Conn_01x02_Male, J27 Conn_01x02_Male, J28 Conn_01x02_Male, J29 Conn_01x02_Male, J3 mic_connector, J30 Conn_01x02_Male, J31 Conn_01x02_Male, J32 Conn_01x02_Male, J33 Conn_01x02_Male, J34 Conn_01x02_Male, J35 Conn_01x02_Male, J36 Conn_01x02_Male, J37 Conn_01x02_Male, J38 Conn_01x02_Male, J39 Conn_01x02_Male, J4 mic_connector, J40 Conn_01x02_Male, J41 Conn_01x02_Male, J42 Conn_01x02_Male, J43 Conn_01x02_Male, J5 mic_connector, J6 mic_connector, J7 mic_connector, J8 mic_connector, J9 SWD_TC2030, U1 STM32F446RETx, U2 DS28E05P

Commit message: reset PCB file to 83b76c623
Parts:
- removed EXP_ORIENTATION: VAL**, audio_shield:EXP_ORIENTATION
- removed the J3 at (149.9, 93.3) (x2)
- added J3: mic_connector, audio_shield:6288_series_8_pos, F.Cu at (149.9, 93.3)
Changed lines of the file:
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@@
     (pad 2 smd rect (at 1 -0.75 270) (size 0.4 1.5) (layers F.Cu F.Paste F.Mask)
       (net 1 +3V0))
-    (pad 6 smd rect (at 3 -0.75 270) (size 0.4 1.5) (layers F.Cu F.Paste F.Mask)
-      (net 62 /I2S3_WS))
-    (pad 8 smd rect (at 3.5 -0.75 270) (size 0.4 1.5) (layers F.Cu F.Paste F.Mask))
-  )
-  (module audio_shield:6288_series_8_pos (layer F.Cu)
-    (at 149.901 93.30092 90)
-    (fp_text reference J3 (at 2.25 3 90) (layer F.SilkS)
-      (effects (font (size 1 1) (thickness 0.15)))
-    )
-    (fp_text value mic_connector (at 1.75 7.5 90) (layer F.Fab)
-      (effects (font (size 1 1) (thickness 0.15)))
-    )
-    (fp_line (start -1.25 0) (end -0.3 0) (layer F.CrtYd) (width 0.12))
-    (fp_poly (pts (xy -1.25 6.1) (xy -3.05 6.1) (xy -3.05 3.9) (xy -1.25 3.9)) (layer F.Cu) (width 0.1))
-    (fp_line (start 3.8 0) (end 4.75 0) (layer F.CrtYd) (width 0.12))
-    (fp_poly (pts (xy 6.55 6.1) (xy 4.75 6.1) (xy 4.75 3.9) (xy 6.55 3.9)) (layer F.Cu) (width 0.1))
-    (fp_line (start -1.25 6.1) (end 4.75 6.1) (layer F.CrtYd) (width 0.12))
-    (fp_line (start -2.5 3.8) (end -2.5 0) (layer F.CrtYd) (width 0.12))
-    (fp_line (start -2.5 0) (end -1.25 0) (layer F.CrtYd) (width 0.12))
-    (fp_line (start 6 3.8) (end 6 0) (layer F.CrtYd) (width 0.12))
-    (fp_line (start 6 0) (end 4.75 0) (layer F.CrtYd) (width 0.12))
-    (fp_line (start 4.75 6.1) (end 6.6 6.1) (layer F.CrtYd) (width 0.12))
-    (fp_line (start 6.6 6.1) (end 6.6 3.8) (layer F.CrtYd) (width 0.12))
-    (fp_line (start 6.6 3.8) (end 6 3.8) (layer F.CrtYd) (width 0.12))
-    (fp_line (start -1.25 6.1) (end -3.1 6.1) (layer F.CrtYd) (width 0.12))
-    (fp_line (start 3.8 0) (end 3.8 -1.6) (layer F.CrtYd) (width 0.12))
-    (fp_line (start 3.8 -1.6) (end -0.3 -1.6) (layer F.CrtYd) (width 0.12))
-    (fp_line (start -0.3 -1.6) (end -0.3 0) (layer F.CrtYd) (width 0.12))
-    (fp_line (start -3.1 6.1) (end -3.1 3.8) (layer F.CrtYd) (width 0.12))
-    (fp_line (start -3.1 3.8) (end -2.5 3.8) (layer F.CrtYd) (width 0.12))
-    (fp_poly (pts (xy 6.55 6.1) (xy 4.75 6.1) (xy 4.75 3.9) (xy 6.55 3.9)) (layer F.Mask) (width 0.1))
-    (fp_poly (pts (xy -1.25 6.1) (xy -3.05 6.1) (xy -3.05 3.9) (xy -1.25 3.9)) (layer F.Mask) (width 0.1))
-    (pad 7 smd rect (at 0 -0.75 90) (size 0.4 1.5) (layers F.Cu F.Paste F.Mask))
-    (pad 1 smd rect (at 0.5 -0.75 90) (size 0.4 1.5) (layers F.Cu F.Paste F.Mask)
-      (net 55 GND))
-    (pad 2 smd rect (at 1 -0.75 90) (size 0.4 1.5) (layers F.Cu F.Paste F.Mask)
-      (net 1 +3V0))
-    (pad 3 smd rect (at 1.5 -0.75 90) (size 0.4 1.5) (layers F.Cu F.Paste F.Mask)
-      (net 57 /I2S1_SD))
-    (pad 4 smd rect (at 2 -0.75 90) (size 0.4 1.5) (layers F.Cu F.Paste F.Mask)
-      (net 58 /I2S1_CK))
-    (pad 5 smd rect (at 2.5 -0.75 90) (size 0.4 1.5) (layers F.Cu F.Paste F.Mask)
-      (net 1 +3V0))
-    (pad 6 smd rect (at 3 -0.75 90) (size 0.4 1.5) (layers F.Cu F.Paste F.Mask)
-      (net 59 /I2S1_WS))
-    (pad 8 smd rect (at 3.5 -0.75 90) (size 0.4 1.5) (layers F.Cu F.Paste F.Mask))
+    (pad 1 smd rect (at 0.5 -0.75 270) (size 0.4 1.5) (layers F.Cu F.Paste F.Mask)
+      (net 54 GND))
+    (pad 7 smd rect (at 0 -0.75 270) (size 0.4 1.5) (layers F.Cu F.Paste F.Mask))
   )
   (module audio_shield:6288_series_8_pos (layer F.Cu)
@@
     (pad 2 smd rect (at 1 -0.75 90) (size 0.4 1.5) (layers F.Cu F.Paste F.Mask)
       (net 1 +3V0))
-    (pad 3 smd rect (at 1.5 -0.75 90) (size 0.4 1.5) (layers F.Cu F.Paste F.Mask)
-      (net 57 /I2S1_SD))
-    (pad 4 smd rect (at 2 -0.75 90) (size 0.4 1.5) (layers F.Cu F.Paste F.Mask)
-      (net 58 /I2S1_CK))
-    (pad 5 smd rect (at 2.5 -0.75 90) (size 0.4 1.5) (layers F.Cu F.Paste F.Mask)
-      (net 55 GND))
-    (pad 6 smd rect (at 3 -0.75 90) (size 0.4 1.5) (layers F.Cu F.Paste F.Mask)
-      (net 59 /I2S1_WS))
-    (pad 8 smd rect (at 3.5 -0.75 90) (size 0.4 1.5) (layers F.Cu F.Paste F.Mask))
-  )
-  (module audio_shield:EXP_ORIENTATION (layer F.Cu)
-    (at 157.7 97)
-    (fp_text reference EXP_ORIENTATION (at 0 1.925) (layer F.SilkS) hide
-      (effects (font (size 1 1) (thickness 0.15)))
-    )
-    (fp_text value VAL** (at 0 3.4) (layer F.SilkS) hide
-      (effects (font (size 1 1) (thickness 0.15)))
-    )
-    (fp_line (start 0 0) (end -0.475 0.475) (layer B.SilkS) (width 0.15))
-    (fp_line (start 0 0) (end 0.475 0.475) (layer B.SilkS) (width 0.15))
-    (fp_line (start 0 0) (end 0.475 -0.475) (layer B.SilkS) (width 0.15))
-    (fp_line (start 0 0) (end -0.475 -0.475) (layer B.SilkS) (width 0.15))
-    (fp_circle (center 0 0) (end 0.7 0.025) (layer B.SilkS) (width 0.15))
-    (fp_line (start 0.7 0) (end 1.8 0) (layer B.SilkS) (width 0.15))
-    (fp_line (start 1.8 0) (end 1.4 -0.35) (layer B.SilkS) (width 0.15))
-    (fp_line (start 1.8 0) (end 1.4 0.35) (layer B.SilkS) (width 0.15))
-    (fp_line (start 1.8 0) (end 1.4 0.35) (layer F.SilkS) (width 0.15))
-    (fp_line (start 1.8 0) (end 1.4 -0.35) (layer F.SilkS) (width 0.15))
-    (fp_line (start 0.7 0) (end 1.8 0) (layer F.SilkS) (width 0.15))
-    (fp_circle (center 0 0) (end 0.7 0.025) (layer F.SilkS) (width 0.15))
-    (fp_circle (center 0 0) (end 0.075 0.025) (layer F.SilkS) (width 0.15))
+    (pad 1 smd rect (at 0.5 -0.75 90) (size 0.4 1.5) (layers F.Cu F.Paste F.Mask)
+      (net 54 GND))
+    (pad 7 smd rect (at 0 -0.75 90) (size 0.4 1.5) (layers F.Cu F.Paste F.Mask))
   )
   (module Jumper:SolderJumper-2_P1.3mm_Bridged_Pad1.0x1.5mm (layer B.Cu)
@@
       (effects (font (size 0.481966 0.481966) (thickness 0.015)) (justify mirror))
     )
+    (fp_line (start 1.325 0.7) (end 1.325 -1.04) (layer B.SilkS) (width 0.127))
+    (fp_line (start 1.325 -1.04) (end -1.325 -1.04) (layer B.SilkS) (width 0.127))
+    (fp_line (start -1.325 -1.04) (end -1.325 0.7) (layer B.SilkS) (width 0.127))
+    (fp_circle (center -1.578 2.232) (end -1.528 2.232) (layer B.SilkS) (width 0.1))
+    (fp_line (start -1.325 2.46) (end 1.325 2.46) (layer B.Fab) (width 0.127))
+    (fp_line (start 1.325 2.46) (end 1.325 -1.04) (layer B.Fab) (width 0.127))
+    (fp_line (start 1.325 -1.04) (end -1.325 -1.04) (layer B.Fab) (width 0.127))
+    (fp_line (start -1.325 -1.04) (end -1.325 2.46) (layer B.Fab) (width 0.127))
+    (fp_line (start -1.651 2.794) (end 1.651 2.794) (layer B.CrtYd) (width 0.05))
+    (fp_line (start 1.651 2.794) (end 1.651 -1.397) (layer B.CrtYd) (width 0.05))
+    (fp_line (start 1.651 -1.397) (end -1.651 -1.397) (layer B.CrtYd) (width 0.05))
+    (fp_line (start -1.651 -1.397) (end -1.651 2.794) (layer B.CrtYd) (width 0.05))
+    (fp_circle (center 0 0) (end 0.456 0) (layer B.Mask) (width 0.912))
+    (fp_poly (pts (xy -0.53 -0.385) (xy -0.43 -0.285) (xy -0.465 -0.23) (xy -0.505 -0.12)
+      (xy -0.51 -0.12) (xy -0.505 -0.11) (xy -0.52 -0.005) (xy -0.523603 0.005)
+      (xy -0.52 0.005) (xy -0.505 0.125) (xy -0.461537 0.224609) (xy -0.426172 0.292666)
+      (xy -0.525 0.39) (xy -0.635 0.505) (xy -0.7 0.41) (xy -0.75 0.31)
+      (xy -0.78 0.22) (xy -0.8 0.14) (xy -0.81 0) (xy -0.796203 -0.160191)
+      (xy -0.75 -0.31) (xy -0.705 -0.4) (xy -0.640309 -0.499766)) (layer B.Paste) (width 0.001))
+    (fp_poly (pts (xy 0.38 -0.53) (xy 0.28 -0.425) (xy 0.23 -0.46) (xy 0.12 -0.5)
+      (xy 0 -0.513603) (xy -0.12 -0.5) (xy -0.224609 -0.461537) (xy -0.287666 -0.426172)
+      (xy -0.385 -0.525) (xy -0.5 -0.64) (xy -0.405 -0.705) (xy -0.31 -0.75)
+      (xy -0.22 -0.78) (xy -0.14 -0.8) (xy 0 -0.81) (xy 0.160191 -0.796203)
+      (xy 0.31 -0.75) (xy 0.425 -0.69) (xy 0.494766 -0.645309)) (layer B.Paste) (width 0.001))
+    (fp_poly (pts (xy 0.53 0.385) (xy 0.425 0.28) (xy 0.46 0.23) (xy 0.5 0.12)
+      (xy 0.513603 0) (xy 0.5 -0.12) (xy 0.461537 -0.224609) (xy 0.421172 -0.282666)
+      (xy 0.52 -0.38) (xy 0.64 -0.5) (xy 0.705 -0.405) (xy 0.75 -0.31)
+      (xy 0.78 -0.23) (xy 0.8 -0.14) (xy 0.81 -0.06) (xy 0.81 0.065)
+      (xy 0.796203 0.160191) (xy 0.78 0.235) (xy 0.75 0.31) (xy 0.705 0.405)
+      (xy 0.640309 0.499766)) (layer B.Paste) (width 0.001))
+    (fp_poly (pts (xy -0.375 0.53) (xy -0.28 0.435) (xy -0.23 0.46) (xy -0.175 0.485)
+      (xy -0.12 0.5) (xy -0.06 0.51) (xy 0 0.513603) (xy 0.12 0.5)
+      (xy 0.224609 0.461537) (xy 0.282666 0.426172) (xy 0.385 0.525) (xy 0.5 0.64)
+      (xy 0.41 0.7) (xy 0.31 0.75) (xy 0.23 0.78) (xy 0.14 0.8)
+      (xy 0 0.81) (xy -0.160191 0.796203) (xy -0.31 0.75) (xy -0.415 0.7)
+      (xy -0.489766 0.645309)) (layer B.Paste) (width 0.001))
     (fp_poly (pts (xy -0.01 0.51) (xy -0.01 0.81) (xy -0.056608 0.808926) (xy -0.098102 0.805661)
       (xy -0.139368 0.800228) (xy -0.180293 0.792643) (xy -0.220765 0.782926) (xy -0.260673 0.771105)
