File: hardware/audio_shield_V3/SPH0645LM4H-B .sch (KiCad schematic (older format))
At the start: 4 parts

Commit message: Update hardware V3 with correct version
Parts:
- C10, C11, MK1, R3: Mount (none) -> placed; Type (none) -> SMD
Changed lines of the file:
@@
 $Descr A4 11693 8268
 encoding utf-8
-Sheet 2 7
+Sheet 5 7
 Title ""
 Date ""
@@
 AR Path="/5F0910F0/5F09357C" Ref="MK7"  Part="1"
 AR Path="/5F0910F8/5F09357C" Ref="MK8"  Part="1"
-F 0 "MK4" H 5000 3667 50  0000 C CNN
+F 0 "MK1" H 5000 3667 50  0000 C CNN
 F 1 "SPH0645LM4H-B" H 5000 3576 50  0000 C CNN
 F 2 "audio_shield:MIC_SPH0645LM4H-B" H 5000 3200 50  0001 L BNN
@@
 F 5 "423-1405-1-ND " H 5000 3200 50  0001 C CNN "Supplier ref."
 F 6 "2.84" H 5000 3200 50  0001 C CNN "Price"
+F 7 "placed" H 5000 3200 50  0001 C CNN "Mount"
+F 8 "SMD" H 5000 3200 50  0001 C CNN "Type"
 	1    5000 3200
 	1    0    0    -1
@@
 AR Path="/5F0910F0/5F09559C" Ref="C23"  Part="1"
 AR Path="/5F0910F8/5F09559C" Ref="C25"  Part="1"
-F 0 "C17" V 6702 2800 50  0000 C CNN
+F 0 "C11" V 6702 2800 50  0000 C CNN
 F 1 "100n" V 6611 2800 50  0000 C CNN
 F 2 "Capacitor_SMD:C_0603_1608Metric" H 6488 2650 50  0001 C CNN
@@
 F 5 "300-86-429" H 6450 2800 50  0001 C CNN "Supplier ref."
 F 6 "0.0093" H 6450 2800 50  0001 C CNN "Price"
+F 7 "placed" H 6450 2800 50  0001 C CNN "Mount"
+F 8 "SMD" H 6450 2800 50  0001 C CNN "Type"
 	1    6450 2800
 	1    0    0    -1
@@
 AR Path="/5F0910F0/5F096212" Ref="C22"  Part="1"
 AR Path="/5F0910F8/5F096212" Ref="C24"  Part="1"
-F 0 "C16" V 6252 2800 50  0000 C CNN
+F 0 "C10" V 6252 2800 50  0000 C CNN
 F 1 "220p" V 6161 2800 50  0000 C CNN
 F 2 "Capacitor_SMD:C_0603_1608Metric" H 6038 2650 50  0001 C CNN
@@
 F 5 "300-86-545" H 6000 2800 50  0001 C CNN "Supplier ref."
 F 6 " 0.0135" H 6000 2800 50  0001 C CNN "Price"
+F 7 "placed" H 6000 2800 50  0001 C CNN "Mount"
+F 8 "SMD" H 6000 2800 50  0001 C CNN "Type"
 	1    6000 2800
 	1    0    0    -1
@@
 AR Path="/5F0910F0/5F0963B1" Ref="R15"  Part="1"
 AR Path="/5F0910F8/5F0963B1" Ref="R17"  Part="1"
-F 0 "R9" H 6070 3246 50  0000 L CNN
+F 0 "R3" H 6070 3246 50  0000 L CNN
 F 1 "68" H 6070 3155 50  0000 L CNN
 F 2 "Resistor_SMD:R_0603_1608Metric" V 5930 3200 50  0001 C CNN
@@
 F 6 "0.283	" H 6000 3200 50  0001 C CNN "Price"
 F 7 "Thick film resistor 0.1W 1%" H 6000 3200 50  0001 C CNN "Description"
+F 8 "placed" H 6000 3200 50  0001 C CNN "Mount"
+F 9 "SMD" H 6000 3200 50  0001 C CNN "Type"
 	1    6000 3200
 	0    -1   -1   0
@@
 AR Path="/5F0910F0/5F099412" Ref="#PWR0143"  Part="1"
 AR Path="/5F0910F8/5F099412" Ref="#PWR0146"  Part="1"
-F 0 "#PWR020" H 6200 2200 50  0001 C CNN
+F 0 "#PWR011" H 6200 2200 50  0001 C CNN
 F 1 "GND" H 6205 2277 50  0000 C CNN
 F 2 "" H 6200 2450 50  0001 C CNN
@@
 AR Path="/5F0910F0/5F09A2A4" Ref="#PWR0144"  Part="1"
 AR Path="/5F0910F8/5F09A2A4" Ref="#PWR0147"  Part="1"
-F 0 "#PWR019" H 5800 3150 50  0001 C CNN
+F 0 "#PWR010" H 5800 3150 50  0001 C CNN
 F 1 "GND" H 5805 3227 50  0000 C CNN
 F 2 "" H 5800 3400 50  0001 C CNN
