File: hardware/audio_shield_V3/leds.sch (KiCad schematic (older format))
At the start: 8 parts

Commit message: Update hardware V3 with correct version
Parts:
- D1, D2, D3, D4, R11, R12, R13, R14: Mount (none) -> placed; Type (none) -> SMD
Connections:
- net GND: now also D1.1 (K), D2.1 (K), D3.1 (K), D4.1 (K); no longer D1.2 (A), D2.2 (A), D3.2 (A), D4.2 (A)
- net at R11.1: now also D1.2 (A); no longer D1.1 (K)
- net at R12.1: now also D2.2 (A); no longer D2.1 (K)
- net at R13.1: now also D3.2 (A); no longer D3.1 (K)
- net at R14.1: now also D4.2 (A); no longer D4.1 (K)
Other:
- moved on the sheet: D1, D2, D3, D4
Changed lines of the file:
@@
 F 6 "0.283	" H 4300 1850 50  0001 C CNN "Price"
 F 7 "Thick film resistor 0.1W 1%" H 4300 1850 50  0001 C CNN "Description"
+F 8 "placed" H 4300 1850 50  0001 C CNN "Mount"
+F 9 "SMD" H 4300 1850 50  0001 C CNN "Type"
 	1    4300 1850
 	0    1    1    0
@@
 F 6 "Distrelec" H 4950 1850 50  0001 C CNN "Supplier"
 F 7 "175-10-257" H 4950 1850 50  0001 C CNN "Supplier ref."
+F 8 "placed" H 4950 1850 50  0001 C CNN "Mount"
+F 9 "SMD" H 4950 1850 50  0001 C CNN "Type"
 	1    4950 1850
-	1    0    0    -1
+	-1   0    0    1
 $EndComp
 $Comp
@@
 F 6 "0.283	" H 4300 2300 50  0001 C CNN "Price"
 F 7 "Thick film resistor 0.1W 1%" H 4300 2300 50  0001 C CNN "Description"
+F 8 "placed" H 4300 2300 50  0001 C CNN "Mount"
+F 9 "SMD" H 4300 2300 50  0001 C CNN "Type"
 	1    4300 2300
 	0    1    1    0
@@
 F 6 "0.283	" H 4300 2700 50  0001 C CNN "Price"
 F 7 "Thick film resistor 0.1W 1%" H 4300 2700 50  0001 C CNN "Description"
+F 8 "placed" H 4300 2700 50  0001 C CNN "Mount"
+F 9 "SMD" H 4300 2700 50  0001 C CNN "Type"
 	1    4300 2700
 	0    1    1    0
@@
 F 6 "Distrelec" H 4950 2700 50  0001 C CNN "Supplier"
 F 7 "175-10-254" H 4950 2700 50  0001 C CNN "Supplier ref."
+F 8 "placed" H 4950 2700 50  0001 C CNN "Mount"
+F 9 "SMD" H 4950 2700 50  0001 C CNN "Type"
 	1    4950 2700
-	1    0    0    -1
+	-1   0    0    1
 $EndComp
 $Comp
@@
 F 6 "0.283	" H 4300 3100 50  0001 C CNN "Price"
 F 7 "Thick film resistor 0.1W 1%" H 4300 3100 50  0001 C CNN "Description"
+F 8 "placed" H 4300 3100 50  0001 C CNN "Mount"
+F 9 "SMD" H 4300 3100 50  0001 C CNN "Type"
 	1    4300 3100
 	0    1    1    0
@@
 F 6 "Distrelec" H 4950 3100 50  0001 C CNN "Supplier"
 F 7 "175-10-254" H 4950 3100 50  0001 C CNN "Supplier ref."
+F 8 "placed" H 4950 3100 50  0001 C CNN "Mount"
+F 9 "SMD" H 4950 3100 50  0001 C CNN "Type"
 	1    4950 3100
-	1    0    0    -1
+	-1   0    0    1
 $EndComp
 Text Notes 5500 1900 0    50   ~ 0
@@
 F 6 "Distrelec" H 4950 2300 50  0001 C CNN "Supplier"
 F 7 "175-10-254" H 4950 2300 50  0001 C CNN "Supplier ref."
+F 8 "placed" H 4950 2300 50  0001 C CNN "Mount"
+F 9 "SMD" H 4950 2300 50  0001 C CNN "Type"
 	1    4950 2300
-	1    0    0    -1
-$EndComp
-Wire Wire Line
+	-1   0    0    1
+$EndComp
+Wire Wire Line
